File: Hardware/CubeX2000.sch (EAGLE design)
At the start: 124 parts, among them IC1 MEGA32-A, IC2 74HC595D, IC3 74HC595D, IC4 74HC595D, IC5 74HC595D, IC6 74HC595D, IC7 74HC595D, IC8 74HC595D, IC9 74HC595D, Q1 16MHz

Commit message: Add files via upload
Parts:
- AVR-ISP: device con-harting-ml:ML10 -> pinhead:PINHD-2X5
- LAYER1, LAYER2, LAYER3, LAYER4, LAYER5, LAYER6, LAYER7, LAYER8, LAYERS: value 22-23-2081 -> (none); device con-molex:22-23-2081 -> pinhead:PINHD-1X8
- Q1: device crystal:CRYSTALHC49U-V -> crystal:CRYSTALHC49S
- RS232: device con-lstb:MA04-1 -> pinhead:PINHD-1X4
Connections:
- net +5V: now also AVR-ISP.9; no longer AVR-ISP.2
- net GND: now also AVR-ISP.10, AVR-ISP.2, AVR-ISP.4, AVR-ISP.6, AVR-ISP.8; no longer AVR-ISP.1, AVR-ISP.3, AVR-ISP.5, AVR-ISP.7, AVR-ISP.9, RESET.P1
- net N$100: now also LAYER5.4; no longer LAYER5-4.S
- net N$101: now also LAYER5.5; no longer LAYER5-5.S
- net N$102: now also LAYER5.6; no longer LAYER5-6.S
- net N$103: now also LAYER5.7; no longer LAYER5-7.S
- net N$104: now also LAYER5.8; no longer LAYER5-8.S
- net N$105: now also LAYER6.1; no longer LAYER6-1.S
- net N$106: now also LAYER6.2; no longer LAYER6-2.S
- net N$107: now also LAYER6.3; no longer LAYER6-3.S
- net N$108: now also LAYER6.4; no longer LAYER6-4.S
- net N$109: now also LAYER6.5; no longer LAYER6-5.S
- net N$110: now also LAYER6.6; no longer LAYER6-6.S
- net N$111: now also LAYER6.7; no longer LAYER6-7.S
- net N$112: now also LAYER6.8; no longer LAYER6-8.S
- net N$113: now also LAYER7.1; no longer LAYER7-1.S
- net N$114: now also LAYER7.2; no longer LAYER7-2.S
- net N$115: now also LAYER7.3; no longer LAYER7-3.S
- net N$116: now also LAYER7.4; no longer LAYER7-4.S
- net N$117: now also LAYER7.5; no longer LAYER7-5.S
- net N$118: now also LAYER7.6; no longer LAYER7-6.S
- net N$119: now also LAYER7.7; no longer LAYER7-7.S
- net N$120: now also LAYER7.8; no longer LAYER7-8.S
- net N$121: now also LAYER8.1; no longer LAYER8-1.S
- net N$122: now also LAYER8.2; no longer LAYER8-2.S
- net N$123: now also LAYER8.3; no longer LAYER8-3.S
- net N$124: now also LAYER8.4; no longer LAYER8-4.S
- net N$125: now also LAYER8.5; no longer LAYER8-5.S
- net N$126: now also LAYER8.6; no longer LAYER8-6.S
- net N$127: now also LAYER8.7; no longer LAYER8-7.S
- net N$128: now also LAYER8.8; no longer LAYER8-8.S
- net N$136: now also AVR-ISP.1; no longer AVR-ISP.10
- net N$137: now also AVR-ISP.5; no longer AVR-ISP.6
- net N$139: now also LAYERS.5; no longer LAYERS-5.S
- net N$141: now also AVR-ISP.3; no longer AVR-ISP.8
- net N$165: now also RS232.2; no longer RS232.4
- net N$168: now also LAYERS.6; no longer LAYERS-6.S
- net N$169: now also AVR-ISP.7; no longer AVR-ISP.4, RESET.S
- net N$170: now also LAYERS.7; no longer LAYERS-7.S
- net N$171: now also LAYERS.8; no longer LAYERS-8.S
- net N$172: now also LAYERS.4; no longer LAYERS-4.S
- net N$173: now also LAYERS.3; no longer LAYERS-3.S
- net N$174: now also LAYERS.2; no longer LAYERS-2.S
- net N$175: now also LAYERS.1; no longer LAYERS-1.S
- net N$65: now also LAYER1.1; no longer LAYER1-1.S
- net N$66: now also LAYER1.2; no longer LAYER1-2.S
- net N$67: now also LAYER1.3; no longer LAYER1-3.S
- net N$68: now also LAYER1.4; no longer LAYER1-4.S
- net N$69: now also LAYER1.5; no longer LAYER1-5.S
- net N$70: now also LAYER1.6; no longer LAYER1-6.S
- net N$71: now also LAYER1.7; no longer LAYER1-7.S
- net N$72: now also LAYER1.8; no longer LAYER1-8.S
- net N$73: now also LAYER2.1; no longer LAYER2-1.S
- net N$74: now also LAYER2.2; no longer LAYER2-2.S
- net N$75: now also LAYER2.3; no longer LAYER2-3.S
- net N$76: now also LAYER2.4; no longer LAYER2-4.S
- net N$77: now also LAYER2.5; no longer LAYER2-5.S
- net N$78: now also LAYER2.6; no longer LAYER2-6.S
- net N$79: now also LAYER2.7; no longer LAYER2-7.S
- net N$80: now also LAYER2.8; no longer LAYER2-8.S
- net N$81: now also LAYER3.1; no longer LAYER3-1.S
- net N$82: now also LAYER3.2; no longer LAYER3-2.S
- net N$83: now also LAYER3.3; no longer LAYER3-3.S
- net N$84: now also LAYER3.4; no longer LAYER3-4.S
- net N$85: now also LAYER3.5; no longer LAYER3-5.S
- net N$86: now also LAYER3.6; no longer LAYER3-6.S
- net N$87: now also LAYER3.7; no longer LAYER3-7.S
- net N$88: now also LAYER3.8; no longer LAYER3-8.S
- net N$89: now also LAYER4.1; no longer LAYER4-1.S
- net N$90: now also LAYER4.2; no longer LAYER4-2.S
- net N$91: now also LAYER4.3; no longer LAYER4-3.S
- net N$92: now also LAYER4.4; no longer LAYER4-4.S
- net N$93: now also LAYER4.5; no longer LAYER4-5.S
- net N$94: now also LAYER4.6; no longer LAYER4-6.S
- net N$95: now also LAYER4.7; no longer LAYER4-7.S
- net N$96: now also LAYER4.8; no longer LAYER4-8.S
- net N$97: now also LAYER5.1; no longer LAYER5-1.S
- net N$98: now also LAYER5.2; no longer LAYER5-2.S
- net N$99: now also LAYER5.3; no longer LAYER5-3.S

Commit message: Add files via upload
Parts:
- removed RESET: (no value), switch-omron:10-XX
- added S1: SKHMPSE010, switch:SKHMPSE010
Connections:
- removed net N$153: C4.1, IC1.GND, IC1.GND1, IC1.GND2, IC1.GND@1
- net GND: now also C4.1, IC1.GND, IC1.GND1, IC1.GND2, IC1.GND@1, S1.1.1, S1.SH; no longer RESET.P
- net N$169: now also S1.2.1; no longer RESET.S1
Changed lines of the file:
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@@
 <?xml version="1.0" encoding="utf-8"?>
 <!DOCTYPE eagle SYSTEM "eagle.dtd">
-<eagle version="7.5.0">
+<eagle version="6.5.0">
 <drawing>
 <settings>
@@
 <grid distance="0.1" unitdist="inch" unit="inch" style="lines" multiple="1" display="no" altdistance="0.01" altunitdist="inch" altunit="inch"/>
 <layers>
-<layer number="1" name="Top" color="4" fill="1" visible="no" active="no"/>
-<layer number="16" name="Bottom" color="1" fill="1" visible="no" active="no"/>
-<layer number="17" name="Pads" color="2" fill="1" visible="no" active="no"/>
-<layer number="18" name="Vias" color="2" fill="1" visible="no" active="no"/>
-<layer number="19" name="Unrouted" color="6" fill="1" visible="no" active="no"/>
-<layer number="20" name="Dimension" color="15" fill="1" visible="no" active="no"/>
-<layer number="21" name="tPlace" color="7" fill="1" visible="no" active="no"/>
-<layer number="22" name="bPlace" color="7" fill="1" visible="no" active="no"/>
-<layer number="23" name="tOrigins" color="15" fill="1" visible="no" active="no"/>
-<layer number="24" name="bOrigins" color="15" fill="1" visible="no" active="no"/>
-<layer number="25" name="tNames" color="7" fill="1" visible="no" active="no"/>
-<layer number="26" name="bNames" color="7" fill="1" visible="no" active="no"/>
-<layer number="27" name="tValues" color="7" fill="1" visible="no" active="no"/>
-<layer number="28" name="bValues" color="7" fill="1" visible="no" active="no"/>
+<layer number="1" name="Top" color="4" fill="1" visible="yes" active="no"/>
+<layer number="16" name="Bottom" color="1" fill="1" visible="yes" active="no"/>
+<layer number="17" name="Pads" color="2" fill="1" visible="yes" active="no"/>
+<layer number="18" name="Vias" color="2" fill="1" visible="yes" active="no"/>
+<layer number="19" name="Unrouted" color="6" fill="1" visible="yes" active="no"/>
+<layer number="20" name="Dimension" color="15" fill="1" visible="yes" active="no"/>
+<layer number="21" name="tPlace" color="7" fill="1" visible="yes" active="no"/>
+<layer number="22" name="bPlace" color="7" fill="1" visible="yes" active="no"/>
+<layer number="23" name="tOrigins" color="15" fill="1" visible="yes" active="no"/>
+<layer number="24" name="bOrigins" color="15" fill="1" visible="yes" active="no"/>
+<layer number="25" name="tNames" color="7" fill="1" visible="yes" active="no"/>
+<layer number="26" name="bNames" color="7" fill="1" visible="yes" active="no"/>
+<layer number="27" name="tValues" color="7" fill="1" visible="yes" active="no"/>
+<layer number="28" name="bValues" color="7" fill="1" visible="yes" active="no"/>
 <layer number="29" name="tStop" color="7" fill="3" visible="no" active="no"/>
 <layer number="30" name="bStop" color="7" fill="6" visible="no" active="no"/>
@@
 <layer number="35" name="tGlue" color="7" fill="4" visible="no" active="no"/>
 <layer number="36" name="bGlue" color="7" fill="5" visible="no" active="no"/>
-<layer number="37" name="tTest" color="7" fill="1" visible="no" active="no"/>
-<layer number="38" name="bTest" color="7" fill="1" visible="no" active="no"/>
+<layer number="37" name="tTest" color="7" fill="1" visible="yes" active="no"/>
+<layer number="38" name="bTest" color="7" fill="1" visible="yes" active="no"/>
 <layer number="39" name="tKeepout" color="4" fill="11" visible="no" active="no"/>
 <layer number="40" name="bKeepout" color="1" fill="11" visible="no" active="no"/>
@@
 <layer number="44" name="Drills" color="7" fill="1" visible="no" active="no"/>
 <layer number="45" name="Holes" color="7" fill="1" visible="no" active="no"/>
-<layer number="46" name="Milling" color="3" fill="1" visible="no" active="no"/>
-<layer number="47" name="Measures" color="7" fill="1" visible="no" active="no"/>
-<layer number="48" name="Document" color="7" fill="1" visible="no" active="no"/>
-<layer number="49" name="Reference" color="7" fill="1" visible="no" active="no"/>
-<layer number="51" name="tDocu" color="7" fill="1" visible="no" active="no"/>
-<layer number="52" name="bDocu" color="7" fill="1" visible="no" active="no"/>
+<layer number="46" name="Milling" color="3" fill="1" visible="yes" active="no"/>
+<layer number="47" name="Measures" color="7" fill="1" visible="yes" active="no"/>
+<layer number="48" name="Document" color="7" fill="1" visible="yes" active="no"/>
+<layer number="49" name="Reference" color="7" fill="1" visible="yes" active="no"/>
+<layer number="51" name="tDocu" color="7" fill="1" visible="yes" active="no"/>
+<layer number="52" name="bDocu" color="7" fill="1" visible="yes" active="no"/>
 <layer number="90" name="Modules" color="5" fill="1" visible="yes" active="yes"/>
 <layer number="91" name="Nets" color="2" fill="1" visible="yes" active="yes"/>
@@
 <part name="SUPPLY17" library="supply2" deviceset="+5V" device=""/>
 <part name="R67" library="resistor" deviceset="R-EU_" device="R1206" value="10K"/>
-<part name="RESET" library="switch-omron" deviceset="10-XX" device=""/>
 <part name="SUPPLY18" library="supply2" deviceset="GND" device=""/>
 <part name="Q1" library="crystal" deviceset="CRYSTAL" device="HC49S" value="16MHz"/>
@@
 <part name="AVR-ISP" library="pinhead" deviceset="PINHD-2X5" device=""/>
 <part name="RS232" library="pinhead" deviceset="PINHD-1X4" device=""/>
+<part name="SUPPLY55" library="supply2" deviceset="GND" device=""/>
+<part name="S1" library="switch" deviceset="SKHMP*E010" device="" technology="S"/>
 </parts>
 <sheets>
@@
 <instance part="SUPPLY17" gate="+5V" x="58.42" y="228.6" rot="R90"/>
 <instance part="R67" gate="G$1" x="73.66" y="228.6"/>
-<instance part="RESET" gate="1" x="73.66" y="236.22" rot="R270"/>
 <instance part="SUPPLY18" gate="GND" x="58.42" y="236.22" rot="R270"/>
 <instance part="Q1" gate="G$1" x="83.82" y="210.82" rot="R90"/>
@@
 <instance part="AVR-ISP" gate="A" x="152.4" y="193.04"/>
 <instance part="RS232" gate="A" x="88.9" y="142.24"/>
+<instance part="SUPPLY55" gate="GND" x="83.82" y="175.26"/>
+<instance part="S1" gate="G$1" x="71.12" y="236.22"/>
 </instances>
 <busses>
@@
 <pinref part="SUPPLY24" gate="GND" pin="GND"/>
 <wire x1="78.74" y1="116.84" x2="93.98" y2="116.84" width="0.1524" layer="91"/>
-</segment>
-<segment>
-<pinref part="RESET" gate="1" pin="P"/>
-<pinref part="SUPPLY18" gate="GND" pin="GND"/>
-<wire x1="68.58" y1="236.22" x2="60.96" y2="236.22" width="0.1524" layer="91"/>
 </segment>
 <segment>
@@
 <pinref part="SUPPLY25" gate="GND" pin="GND"/>
 <wire x1="81.28" y1="147.32" x2="81.28" y2="149.86" width="0.1524" layer="91"/>
+</segment>
+<segment>
+<pinref part="IC1" gate="G$1" pin="GND1"/>
+<wire x1="88.9" y1="182.88" x2="83.82" y2="182.88" width="0.1524" layer="91"/>
+<wire x1="83.82" y1="182.88" x2="83.82" y2="180.34" width="0.1524" layer="91"/>
+<pinref part="IC1" gate="G$1" pin="GND2"/>
+<wire x1="83.82" y1="180.34" x2="83.82" y2="177.8" width="0.1524" layer="91"/>
+<wire x1="88.9" y1="177.8" x2="83.82" y2="177.8" width="0.1524" layer="91"/>
+<pinref part="IC1" gate="G$1" pin="GND"/>
+<wire x1="88.9" y1="180.34" x2="83.82" y2="180.34" width="0.1524" layer="91"/>
+<junction x="83.82" y="180.34"/>
+<wire x1="83.82" y1="182.88" x2="83.82" y2="198.12" width="0.1524" layer="91"/>
+<junction x="83.82" y="182.88"/>
+<pinref part="IC1" gate="G$1" pin="GND@1"/>
+<wire x1="83.82" y1="198.12" x2="88.9" y2="198.12" width="0.1524" layer="91"/>
+<pinref part="C4" gate="G$1" pin="1"/>
+<wire x1="83.82" y1="182.88" x2="76.2" y2="182.88" width="0.1524" layer="91"/>
+<wire x1="76.2" y1="182.88" x2="76.2" y2="187.96" width="0.1524" layer="91"/>
+<pinref part="SUPPLY55" gate="GND" pin="GND"/>
+<junction x="83.82" y="177.8"/>
+</segment>
+<segment>
+<pinref part="SUPPLY18" gate="GND" pin="GND"/>
+<pinref part="S1" gate="G$1" pin="1.1"/>
+<wire x1="60.96" y1="236.22" x2="66.04" y2="236.22" width="0.1524" layer="91"/>
+<pinref part="S1" gate="G$1" pin="SH"/>
+<wire x1="66.04" y1="231.14" x2="66.04" y2="236.22" width="0.1524" layer="91"/>
+<junction x="66.04" y="236.22"/>
 </segment>
 </net>
@@
 </segment>
 </net>
-<net name="N$153" class="0">
-<segment>
-<pinref part="IC1" gate="G$1" pin="GND1"/>
-<wire x1="88.9" y1="182.88" x2="83.82" y2="182.88" width="0.1524" layer="91"/>
-<wire x1="83.82" y1="182.88" x2="83.82" y2="180.34" width="0.1524" layer="91"/>
-<pinref part="IC1" gate="G$1" pin="GND2"/>
-<wire x1="83.82" y1="180.34" x2="83.82" y2="177.8" width="0.1524" layer="91"/>
-<wire x1="88.9" y1="177.8" x2="83.82" y2="177.8" width="0.1524" layer="91"/>
-<pinref part="IC1" gate="G$1" pin="GND"/>
-<wire x1="88.9" y1="180.34" x2="83.82" y2="180.34" width="0.1524" layer="91"/>
-<junction x="83.82" y="180.34"/>
-<wire x1="83.82" y1="182.88" x2="83.82" y2="198.12" width="0.1524" layer="91"/>
-<junction x="83.82" y="182.88"/>
-<pinref part="IC1" gate="G$1" pin="GND@1"/>
-<wire x1="83.82" y1="198.12" x2="88.9" y2="198.12" width="0.1524" layer="91"/>
-<pinref part="C4" gate="G$1" pin="1"/>
-<wire x1="83.82" y1="182.88" x2="76.2" y2="182.88" width="0.1524" layer="91"/>
-<wire x1="76.2" y1="182.88" x2="76.2" y2="187.96" width="0.1524" layer="91"/>
-</segment>
-</net>
 <net name="N$156" class="0">
 <segment>
@@
 <net name="N$169" class="0">
 <segment>
-<pinref part="RESET" gate="1" pin="S1"/>
 <wire x1="149.86" y1="190.5" x2="142.24" y2="190.5" width="0.1524" layer="91"/>
 <wire x1="142.24" y1="190.5" x2="142.24" y2="228.6" width="0.1524" layer="91"/>
@@
 <wire x1="78.74" y1="228.6" x2="83.82" y2="228.6" width="0.1524" layer="91"/>
 <junction x="83.82" y="228.6"/>
-<wire x1="78.74" y1="233.68" x2="83.82" y2="233.68" width="0.1524" layer="91"/>
 <wire x1="83.82" y1="233.68" x2="83.82" y2="228.6" width="0.1524" layer="91"/>
 <pinref part="C19" gate="G$1" pin="2"/>
+<pinref part="AVR-ISP" gate="A" pin="7"/>
+<pinref part="S1" gate="G$1" pin="2.1"/>
+<wire x1="78.74" y1="236.22" x2="83.82" y2="236.22" width="0.1524" layer="91"/>
+<wire x1="83.82" y1="236.22" x2="83.82" y2="233.68" width="0.1524" layer="91"/>
 <junction x="83.82" y="233.68"/>
-<pinref part="AVR-ISP" gate="A" pin="7"/>
-</segment>
-</net>
+</segment>
+</net>

Commit message: Add files via upload
Parts:
- renumbered LAYER1 to ROW1, LAYER2 to ROW2, LAYER3 to ROW3, LAYER4 to ROW4, LAYER5 to ROW5, LAYER6 to ROW6, LAYER7 to ROW7, LAYER8 to ROW8
Connections:
- net GND: now also S1.1.2
Other:
- moved on the sheet: S1

Commit message: Add files via upload
Parts:
- removed C16: 100nf, resistor:C-EUC1206
- removed C5, C6, C7: 1uF, resistor:C-EUC1206
- removed RS232: (no value), pinhead:PINHD-1X4
- removed U$9: MAX232D, maxim:MAX232D
- added KONWERTER-USB: (no value), pinhead:PINHD-1X5
Connections:
- removed net N$144: C6.2, U$9G$1.C1+
- removed net N$145: C6.1, U$9G$1.C1-
- removed net N$146: C5.2, U$9G$1.C2+
- removed net N$147: C5.1, U$9G$1.C2-
- removed net N$148: RS232.3, U$9G$1.R1IN
- removed net N$154: IC1.(TXD)PD1, U$9G$1.R1OUT
- removed net N$155: IC1.(RXD)PD0, U$9G$1.T1IN
- removed net N$165: RS232.2, U$9G$1.T1OUT
- net +5V: now also KONWERTER-USB.1; no longer C16.2, U$9G$2.VCC
- net GND: now also KONWERTER-USB.5; no longer C16.1, RS232.1, U$9G$2.GND
- net N$142: now also IC1.(RXD)PD0, KONWERTER-USB.4; no longer C7.2, U$9G$1.V+
- net N$143: now also IC1.(TXD)PD1, KONWERTER-USB.3; no longer C7.1, U$9G$1.V-
- net N$169: now also KONWERTER-USB.2
