File: Hardware/CubeX2000.brd (EAGLE design)
At the start: 100 x 80 mm, 123 parts, among them IC1 MEGA32-A, IC10 MAX232, IC2 74HC595D, IC3 74HC595D, IC4 74HC595D, IC5 74HC595D, IC6 74HC595D, IC7 74HC595D, IC8 74HC595D, IC9 74HC595D, Q1 16MHz

Commit message: Add files via upload
Parts:
- removed IC10: MAX232, maxim:DIL16
- added C19: 100nf, resistor:C1206
- added U$9: MAX232D, maxim:SO16
- moved R40 88.8 mm to (95.9, 44.5), flipped to the bottom
- moved R1 87.4 mm to (10.4, 70.7), flipped to the bottom
- moved R32 85.3 mm to (96.8, 70.7), flipped to the bottom
- moved R57 84.0 mm to (9.53, 44.5), flipped to the bottom
- moved R39 83.7 mm to (93.3, 44.5), flipped to the bottom
- moved R2 82.3 mm to (13.0, 70.7), flipped to the bottom
- moved R31 80.3 mm to (94.2, 70.7), flipped to the bottom
- moved R58 78.9 mm to (12.1, 44.5), flipped to the bottom
- moved R38 78.6 mm to (90.8, 44.5), flipped to the bottom
- moved R3 77.2 mm to (15.5, 70.7), flipped to the bottom
- moved R30 75.2 mm to (91.7, 70.7), flipped to the bottom
- moved R59 73.8 mm to (14.6, 44.5), flipped to the bottom
- moved R37 73.5 mm to (88.3, 44.5), flipped to the bottom
- moved R4 72.1 mm to (18.0, 70.7), flipped to the bottom
- moved LAYER5 71.0 mm to (87.0, 49.7), turned to 0 degrees
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Connections:
- removed net N$158: C5.2, IC10.5
- removed net N$159: C5.1, IC10.4
- removed net N$160: C6.2, IC10.3
- removed net N$161: C6.1, IC10.1
- removed net N$162: C7.2, IC10.6
- removed net N$163: C7.1, IC10.2
- new net N$142: C7.2, U$9.2
- new net N$143: C7.1, U$9.6
- new net N$144: C6.2, U$9.1
- new net N$145: C6.1, U$9.3
- new net N$146: C5.2, U$9.4
- new net N$147: C5.1, U$9.5
- net +5V: now also U$9.16; no longer IC10.16
- net GND: now also C19.1, U$9.15; no longer IC10.15
- net N$154: now also U$9.12; no longer IC10.12
- net N$155: now also U$9.11; no longer IC10.11
- net N$164: now also U$9.13; no longer IC10.13
- net N$165: now also U$9.14; no longer IC10.14
- net N$169: now also C19.2
Routing:
- net GND: track 31.8 -> 489.9 mm
- net +5V: track 29.2 -> 220.8 mm, vias 0 -> 12
- net N$138: track 180.8 -> 290.7 mm, vias 0 -> 4
- net N$136: track 181.2 -> 273.3 mm, vias 0 -> 2
- net N$135: track 0.00 -> 43.7 mm, vias 0 -> 2
- net N$129: track 0.00 -> 39.9 mm, vias 0 -> 2
- net N$130: track 0.00 -> 39.5 mm, vias 0 -> 2
- net N$131: track 0.00 -> 35.3 mm, vias 0 -> 2
- net N$140: track 180.2 -> 210.0 mm
- net N$134: track 0.00 -> 20.0 mm, vias 0 -> 2
- net N$132: track 0.00 -> 19.5 mm, vias 0 -> 2
- net N$133: track 0.00 -> 19.5 mm, vias 0 -> 2
- net N$96: track 5.08 -> 0.00 mm
- net N$75: track 5.08 -> 0.00 mm
- net N$99: track 4.93 -> 0.00 mm
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
Commit message: Add files via upload
Parts:
- moved U$4 28.7 mm to (68.3, 13.5), turned to 180 degrees
- moved RESET 27.2 mm to (34.7, 6.99)
- moved C19 23.1 mm to (40.3, 23.6)
- moved U$1 23.1 mm to (71.5, 10.0), turned to 180 degrees
- moved U$8 21.1 mm to (82.3, 18.0)
- moved U$5 19.0 mm to (75.3, 10.0), turned to 180 degrees
- moved U$6 18.7 mm to (82.3, 14.2)
- moved C3 18.1 mm to (66.4, 8.13), turned to 90 degrees
- moved U$2 16.3 mm to (79.2, 10.0), turned to 180 degrees
- moved U$3 15.9 mm to (83.2, 10.0), turned to 180 degrees
- moved AVR-ISP 15.7 mm to (28.8, 17.9)
- moved IC1 14.8 mm to (58.9, 15.6)
- moved C4 14.2 mm to (59.1, 6.86), turned to 180 degrees
- moved C1 14.0 mm to (46.9, 17.1)
- moved C2 14.0 mm to (46.9, 22.0)
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Routing:
- net +5V: track 220.8 -> 316.7 mm, vias 12 -> 20
- net GND: track 489.9 -> 569.5 mm
- net N$140: track 210.0 -> 281.9 mm, vias 0 -> 4
- net N$169: track 0.00 -> 52.5 mm, vias 0 -> 2
- net N$155: track 0.00 -> 48.3 mm
- net N$154: track 0.00 -> 46.9 mm
- net N$137: track 0.00 -> 34.0 mm, vias 0 -> 2
- net N$141: track 0.00 -> 33.2 mm, vias 0 -> 2
- net N$171: track 0.00 -> 30.9 mm
- net N$153: track 0.00 -> 26.7 mm
- net LAYERS2: track 0.00 -> 25.2 mm
- net LAYERS1: track 0.00 -> 25.2 mm
- net LAYERS3: track 0.00 -> 24.8 mm
- net N$170: track 0.00 -> 23.9 mm
- net LAYERS4: track 0.00 -> 23.6 mm
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
Commit message: Add files via upload
Parts:
- AVR-ISP: device con-harting-ml:ML10 -> pinhead:2X05
- LAYER1, LAYER2, LAYER3, LAYER4, LAYER5, LAYER6, LAYER7, LAYER8, LAYERS: value 22-23-2081 -> (none); device con-molex:22-23-2081 -> pinhead:1X08
- Q1: device crystal:HC49U-V -> crystal:HC49/S
- RS232: device con-lstb:MA04-1 -> pinhead:1X04
- moved LED1 50.9 mm to (53.5, 19.7)
- moved LED2 48.1 mm to (50.7, 22.4), turned to 180 degrees
- moved R68 45.6 mm to (53.5, 17.3), turned to 180 degrees
- moved R69 41.4 mm to (49.3, 18.8), turned to 90 degrees
- moved C7 21.1 mm to (2.16, 15.4), turned to 270 degrees
- moved U$7 19.9 mm to (97.8, 9.53), turned to 180 degrees
- moved C5 18.3 mm to (3.56, 19.2), turned to 180 degrees
- moved C1 16.4 mm to (30.6, 15.4)
- moved C4 15.5 mm to (44.2, 2.20), turned to 225 degrees
- moved Q1 15.0 mm to (34.7, 15.6), turned to 225 degrees
- moved AVR-ISP 14.6 mm to (29.6, 3.30)
- moved C2 14.5 mm to (32.9, 18.2)
- moved C19 14.4 mm to (28.3, 15.5), turned to 270 degrees
- moved U$8 14.0 mm to (93.5, 9.53), turned to 180 degrees
- moved RESET 13.2 mm to (23.5, 14.0), turned to 270 degrees
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Connections:
- net +5V: now also AVR-ISP.9; no longer AVR-ISP.2
- net GND: now also AVR-ISP.10, AVR-ISP.2, AVR-ISP.4, AVR-ISP.6, AVR-ISP.8; no longer AVR-ISP.1, AVR-ISP.3, AVR-ISP.5, AVR-ISP.7, AVR-ISP.9, RESET.4
- net N$136: now also AVR-ISP.1; no longer AVR-ISP.10
- net N$137: now also AVR-ISP.5; no longer AVR-ISP.6
- net N$141: now also AVR-ISP.3; no longer AVR-ISP.8
- net N$165: now also RS232.2; no longer RS232.4
- net N$169: now also AVR-ISP.7; no longer AVR-ISP.4, RESET.1
Routing:
- net GND: track 569.5 -> 685.7 mm, vias 0 -> 6
- net N$136: track 273.3 -> 306.4 mm, vias 2 -> 4
- net +5V: track 316.7 -> 348.1 mm, vias 20 -> 16
- net LAYERS1: track 25.2 -> 55.9 mm, vias 0 -> 2
- net LAYERS2: track 25.2 -> 50.9 mm, vias 0 -> 2
- net N$153: track 26.7 -> 3.79 mm
- net N$171: track 30.9 -> 8.48 mm
- net LAYERS3: track 24.8 -> 45.1 mm, vias 0 -> 2
- net N$169: track 52.5 -> 32.5 mm, vias 2 -> 0
- net LAYERS5: track 17.3 -> 36.1 mm, vias 0 -> 2
- net LAYERS6: track 14.6 -> 32.7 mm, vias 0 -> 2
- net LAYERS7: track 11.4 -> 28.2 mm, vias 0 -> 2
- net LAYERS4: track 23.6 -> 40.4 mm, vias 0 -> 2
- net N$170: track 23.9 -> 7.90 mm
- net N$137: track 34.0 -> 18.8 mm
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
Commit message: Add files via upload
Routing:
- net N$140: track 283.0 -> 308.6 mm, vias 4 -> 6
- net GND: track 685.7 -> 701.1 mm
- net N$129: track 41.0 -> 38.6 mm
- net N$136: track 306.4 -> 308.5 mm
- net N$137: track 18.8 -> 18.3 mm
Changed lines of the file:
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@@
 <wire x1="14.3764" y1="15.494" x2="12.827" y2="15.494" width="0.4064" layer="16"/>
 <wire x1="12.827" y1="15.494" x2="12.319" y2="14.986" width="0.4064" layer="16"/>
+<wire x1="12.319" y1="9.779" x2="12.573" y2="9.779" width="0.4064" layer="16"/>
+<wire x1="12.573" y1="9.779" x2="20.32" y2="2.032" width="0.4064" layer="16"/>
+<wire x1="20.32" y1="2.032" x2="24.511" y2="2.032" width="0.4064" layer="16"/>
+<wire x1="69.469" y1="64.008" x2="69.469" y2="64.9224" width="0" layer="19" extent="16-16"/>
 <wire x1="12.319" y1="14.986" x2="12.319" y2="9.779" width="0.4064" layer="16"/>
-<wire x1="69.469" y1="64.008" x2="69.469" y2="64.9224" width="0" layer="19" extent="16-16"/>
-<wire x1="23.5712" y1="19.558" x2="17.78" y2="32.4866" width="0" layer="19" extent="16-16"/>
 </signal>
 <signal name="N$129">
 <contactref element="IC8" pad="9"/>
 <contactref element="IC9" pad="14"/>
-<wire x1="16.51" y1="32.4866" x2="16.383" y2="26.67" width="0.4064" layer="16"/>
-<via x="16.383" y="26.67" extent="1-16" drill="0.6" diameter="1.778"/>
-<wire x1="16.383" y1="26.67" x2="45.72" y2="26.67" width="0.4064" layer="1"/>
-<via x="45.72" y="26.67" extent="1-16" drill="0.6" diameter="1.778"/>
-<wire x1="45.72" y1="32.4866" x2="45.72" y2="26.67" width="0.4064" layer="16"/>
+<wire x1="16.51" y1="32.4866" x2="16.256" y2="27.94" width="0.4064" layer="16"/>
+<via x="16.256" y="27.94" extent="1-16" drill="0.6" diameter="1.778"/>
+<wire x1="16.256" y1="27.94" x2="45.72" y2="27.94" width="0.4064" layer="1"/>
+<via x="45.72" y="27.94" extent="1-16" drill="0.6" diameter="1.778"/>
+<wire x1="45.72" y1="32.4866" x2="45.72" y2="27.94" width="0.4064" layer="16"/>
 </signal>
 <signal name="N$130">
@@
 <wire x1="20.32" y1="30.099" x2="20.32" y2="32.4866" width="0.4064" layer="16"/>
 <contactref element="AVR-ISP" pad="1"/>
-<wire x1="34.671" y1="4.572" x2="34.671" y2="6.604" width="0.4064" layer="16"/>
-<wire x1="34.671" y1="6.604" x2="40.513" y2="12.446" width="0.4064" layer="16"/>
-<wire x1="40.513" y1="12.446" x2="40.64" y2="12.446" width="0.4064" layer="16"/>
+<wire x1="34.671" y1="4.572" x2="34.798" y2="10.414" width="0.4064" layer="16"/>
+<wire x1="34.798" y1="10.414" x2="36.957" y2="12.446" width="0.4064" layer="16"/>
+<wire x1="36.957" y1="12.446" x2="40.64" y2="12.446" width="0.4064" layer="16"/>
 <wire x1="43.218615625" y1="12.446" x2="44.902890625" y2="10.761725" width="0.4064" layer="16"/>
 <wire x1="43.218615625" y1="12.446" x2="40.64" y2="12.446" width="0.4064" layer="16"/>
@@
 <contactref element="IC1" pad="1"/>
 <contactref element="AVR-ISP" pad="5"/>
-<wire x1="29.591" y1="4.572" x2="29.591" y2="8.89" width="0.4064" layer="16"/>
-<via x="29.591" y="8.89" extent="1-16" drill="0.6" diameter="1.4224"/>
-<wire x1="29.591" y1="8.89" x2="42.164" y2="8.89" width="0.4064" layer="1"/>
-<via x="42.164" y="8.89" extent="1-16" drill="0.6" diameter="1.4224"/>
-<wire x1="42.164" y1="8.89" x2="43.03116875" y2="8.89" width="0.4064" layer="16"/>
+<wire x1="29.591" y1="4.572" x2="29.591" y2="7.874" width="0.4064" layer="16"/>
+<via x="29.591" y="7.874" extent="1-16" drill="0.6" diameter="1.4224"/>
+<wire x1="29.591" y1="7.874" x2="42.164" y2="7.874" width="0.4064" layer="1"/>
+<via x="42.164" y="7.874" extent="1-16" drill="0.6" diameter="1.4224"/>
+<wire x1="42.164" y1="7.874" x2="43.03116875" y2="8.89" width="0.4064" layer="16"/>
 <wire x1="43.03116875" y1="8.89" x2="43.771521875" y2="9.630353125" width="0.4064" layer="16"/>
-<wire x1="29.591" y1="8.89" x2="17.399" y2="58.7756" width="0" layer="19" extent="1-16"/>
+<wire x1="29.591" y1="7.874" x2="17.399" y2="58.7756" width="0" layer="19" extent="1-16"/>
 </signal>
 <signal name="N$140">
@@
 <wire x1="41.91" y1="32.4866" x2="41.91" y2="29.083" width="0.4064" layer="16"/>
 <wire x1="41.91" y1="29.083" x2="40.386" y2="27.051" width="0.4064" layer="16"/>
-<wire x1="40.386" y1="27.051" x2="32.893" y2="27.051" width="0.4064" layer="16"/>
+<wire x1="37.846" y1="27.051" x2="32.893" y2="27.051" width="0.4064" layer="16"/>
 <wire x1="29.21" y1="36.195" x2="21.209" y2="36.195" width="0.4064" layer="16"/>
 <wire x1="21.209" y1="36.195" x2="19.177" y2="33.909" width="0.4064" layer="16"/>
@@
 <wire x1="42.799" y1="58.7756" x2="42.799" y2="58.039" width="0" layer="19" extent="16-16"/>
 <wire x1="87.63" y1="31.623" x2="87.884" y2="32.2326" width="0" layer="19" extent="16-16"/>
-<wire x1="43.771521875" y1="7.08476875" x2="40.386" y2="27.051" width="0" layer="19" extent="16-16"/>
+<wire x1="40.386" y1="27.051" x2="37.846" y2="27.051" width="0.4064" layer="16"/>
+<wire x1="37.846" y1="27.051" x2="37.846" y2="26.162" width="0.4064" layer="16"/>
+<via x="37.846" y="26.162" extent="1-16" drill="0.6"/>
+<wire x1="37.846" y1="26.162" x2="37.846" y2="10.795" width="0.4064" layer="1"/>
+<via x="37.846" y="10.795" extent="1-16" drill="0.6"/>
+<wire x1="37.846" y1="10.795" x2="37.846" y2="8.382" width="0.4064" layer="16"/>
+<wire x1="37.846" y1="8.382" x2="39.751" y2="6.477" width="0.4064" layer="16"/>
+<wire x1="39.751" y1="6.477" x2="43.163753125" y2="6.477" width="0.4064" layer="16"/>
+<wire x1="43.163753125" y1="6.477" x2="43.771521875" y2="7.08476875" width="0.4064" layer="16"/>
 </signal>
 <signal name="N$141">
 <contactref element="IC1" pad="2"/>
 <contactref element="AVR-ISP" pad="3"/>
-<wire x1="32.131" y1="4.572" x2="32.131" y2="10.922" width="0.4064" layer="16"/>
-<via x="32.131" y="10.922" extent="1-16" drill="0.6" diameter="1.4224"/>
-<wire x1="32.131" y1="10.922" x2="41.656" y2="10.922" width="0.4064" layer="1"/>
-<via x="41.656" y="10.922" extent="1-16" drill="0.6" diameter="1.4224"/>
-<wire x1="41.656" y1="10.922" x2="43.307" y2="10.922" width="0.4064" layer="16"/>
-<wire x1="43.307" y1="10.922" x2="44.33720625" y2="10.1960375" width="0.4064" layer="16"/>
+<wire x1="32.131" y1="4.572" x2="32.131" y2="9.525" width="0.4064" layer="16"/>
+<via x="32.131" y="9.525" extent="1-16" drill="0.6" diameter="1.4224"/>
+<wire x1="32.131" y1="9.525" x2="41.021" y2="9.525" width="0.4064" layer="1"/>
+<via x="41.021" y="9.525" extent="1-16" drill="0.6" diameter="1.4224"/>
+<wire x1="41.021" y1="9.525" x2="43.053" y2="11.43" width="0.4064" layer="16"/>
+<wire x1="43.053" y1="11.43" x2="44.33720625" y2="10.1960375" width="0.4064" layer="16"/>
 </signal>
 <signal name="+5V">

Commit message: Add files via upload
Parts:
- moved C3 1.02 mm to (61.6, 1.91)
Routing:
- net N$137: track 18.3 -> 98.2 mm, vias 2 -> 6
- net N$136: track 308.5 -> 271.3 mm, vias 4 -> 8
- net N$153: track 3.79 -> 20.8 mm
- net N$140: track 308.6 -> 318.6 mm
- net +5V: track 348.1 -> 354.3 mm, vias 16 -> 20
- net N$138: track 298.3 -> 300.6 mm
- net N$135: track 40.5 -> 42.5 mm, vias 2 -> 4
- net N$152: track 7.41 -> 8.79 mm
- net N$1: track 13.7 -> 12.9 mm

Commit message: Add files via upload
Parts:
- removed RESET: (no value), switch-omron:B3F-10XX
- added S1: SKHMPSE010, switch:SKHMPXE010
- moved AVR-ISP 1.91 mm to (29.6, 1.40)
- moved IC8 1.42 mm to (42.5, 34.9)
- moved IC9 1.42 mm to (19.7, 34.9)
- moved IC6 1.42 mm to (88.3, 34.9)
- moved IC7 1.42 mm to (65.4, 34.9)
- moved IC2 1.27 mm to (20.6, 61.8)
- moved IC3 1.27 mm to (43.4, 61.8)
- moved IC4 1.27 mm to (66.3, 61.8)
- moved IC5 1.27 mm to (89.2, 61.8)
- moved LED1 0.63 mm to (53.5, 19.1)
- moved LED2 0.51 mm to (50.7, 21.8)
- moved R68 0.38 mm to (53.5, 16.9)
- moved R69 0.38 mm to (49.3, 18.4)
Connections:
- removed net N$153: C4.1, IC1.18, IC1.28, IC1.39, IC1.6
- net GND: now also C4.1, IC1.18, IC1.28, IC1.39, IC1.6, S1.1, S1.5; no longer RESET.3
- net N$169: now also S1.3; no longer RESET.2
Routing:
- net GND: track 701.2 -> 764.4 mm, vias 6 -> 0
- net +5V: track 354.3 -> 391.1 mm, vias 20 -> 26
- net N$138: track 300.6 -> 275.6 mm
- net N$153: track 20.8 -> 0.00 mm
- net N$130: track 34.2 -> 46.1 mm
- net N$135: track 42.5 -> 49.9 mm
- net N$140: track 318.6 -> 325.1 mm
- net N$137: track 98.2 -> 102.7 mm
- net N$141: track 18.4 -> 20.4 mm
- net N$58: track 5.18 -> 7.03 mm
- net N$42: track 5.18 -> 6.88 mm
- net N$26: track 5.18 -> 6.62 mm
- net N$15: track 7.13 -> 5.71 mm
- net N$50: track 5.18 -> 6.58 mm
- net N$23: track 7.05 -> 5.71 mm
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Other:
- board size 100 x 80 mm -> 106.7 x 83.9 mm
- board text added: "CubeX2000"
- board text added: "Marcin Przadka"

Commit message: Add files via upload
Parts:
- renumbered LAYER1 to ROW1, LAYER2 to ROW2, LAYER3 to ROW3, LAYER4 to ROW4, LAYER5 to ROW5, LAYER6 to ROW6, LAYER7 to ROW7, LAYER8 to ROW8
Connections:
- net GND: now also S1.2

Commit message: Add files via upload
Parts:
- removed C16: 100nf, resistor:C1206
- removed C5, C6, C7: 1uF, resistor:C1206
- removed RS232: (no value), pinhead:1X04
- removed U$9: MAX232D, maxim:SO16
- added KONWERTER-USB: (no value), pinhead:1X05
- moved S1 3.72 mm to (20.8, 11.8)
- moved ROW6 0.38 mm to (64.1, 48.6)
- moved ROW7 0.13 mm to (41.3, 48.8)
- moved ROW3 0.13 mm to (65.0, 75.1)
Connections:
- removed net N$144: C6.2, U$9.1
- removed net N$145: C6.1, U$9.3
- removed net N$146: C5.2, U$9.4
- removed net N$147: C5.1, U$9.5
- removed net N$148: RS232.3, U$9.13
- removed net N$154: IC1.10, U$9.12
- removed net N$155: IC1.9, U$9.11
- removed net N$165: RS232.2, U$9.14
- net +5V: now also KONWERTER-USB.1; no longer C16.2, U$9.16
- net GND: now also KONWERTER-USB.5; no longer C16.1, RS232.1, U$9.15
- net N$142: now also IC1.9, KONWERTER-USB.4; no longer C7.2, U$9.2
- net N$143: now also IC1.10, KONWERTER-USB.3; no longer C7.1, U$9.6
- net N$169: now also KONWERTER-USB.2
Routing:
- net GND: track 764.4 -> 147.3 mm
- net N$154: track 39.1 -> 0.00 mm
- net N$155: track 36.9 -> 0.00 mm, vias 2 -> 0
- net N$142: track 6.85 -> 32.3 mm
- net N$169: track 32.8 -> 55.8 mm
- net N$143: track 13.6 -> 36.1 mm
- net N$138: track 275.6 -> 261.3 mm
- net N$148: track 13.3 -> 0.00 mm
- net N$165: track 10.1 -> 0.00 mm
- net +5V: track 391.1 -> 400.6 mm
- net N$147: track 8.04 -> 0.00 mm
- net N$146: track 3.75 -> 0.00 mm
- net N$144: track 3.66 -> 0.00 mm
- net N$145: track 3.41 -> 0.00 mm
- net N$137: track 102.7 -> 99.4 mm
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- added copper zone on layer 16, net GND
Other:
- board text added: "Marcin Przadka.net"
- board text removed: "Marcin Przadka"
